File: Electronics/Motors/Motor Driver/Motor Driver Board/Motor Driver Board.kicad_sch (KiCad schematic)
At the start: 4 parts

Commit message: PCB Schematic progress
Other:
- sheet Motor Driver renamed Motor Drivers
Changed lines of the file:
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@@
     (stroke (width 0.1524) (type solid))
     (fill (color 0 0 194 1.0000))
-    (property "Sheetname" "Motor Driver" (at 83.82 37.3884 0)
+    (property "Sheetname" "Motor Drivers" (at 83.82 37.3884 0)
       (effects (font (size 1.27 1.27)) (justify left bottom))
     )
