File: Electronics/Motors/Motor Driver/Motor Driver Board/motor_driver.kicad_sch (KiCad schematic)
At the start: 52 parts, among them J4 XT60PW-F, J5 XT60PW-F, J6 XT60PW-F, J7 XT60PW-M, T1 NVMFS4C05NT1G, T10 NVMFS4C05NT1G, T11 NVMFS4C05NT1G, T12 NVMFS4C05NT1G, T2 NVMFS4C05NT1G, T3 NVMFS4C05NT1G, T4 NVMFS4C05NT1G, T5 NVMFS4C05NT1G, T6 NVMFS4C05NT1G, T7 NVMFS4C05NT1G, T8 NVMFS4C05NT1G, T9 NVMFS4C05NT1G, U2 DRV8701ERGER, U3 DRV8701ERGER, U4 DRV8701ERGER

Commit message: PCB Schematic progress
Parts:
- C46, C48, C50: footprint (none) -> Capacitor_SMD:CP_Elec_6.3x7.7
Other:
- note added: "16V Cap"
Changed lines of the file:
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@@
     (effects (font (size 2.54 2.54)) (justify left bottom))
+  )
+  (text "16V Cap" (at 139.7 120.65 0)
+    (effects (font (size 1.27 1.27)) (justify left bottom))
+  )
+  (text "16V Cap" (at 308.61 120.65 0)
+    (effects (font (size 1.27 1.27)) (justify left bottom))
   )
   (text "Motor 2" (at 224.79 40.64 0)
@@
   (text "Motor 1" (at 57.15 40.64 0)
     (effects (font (size 2.54 2.54)) (justify left bottom))
+  )
+  (text "16V Cap" (at 135.89 241.3 0)
+    (effects (font (size 1.27 1.27)) (justify left bottom))
   )
   (text "Motor 3" (at 55.88 160.02 0)
@@
       (effects (font (size 1.27 1.27)) (justify right))
     )
-    (property "Footprint" "" (at 173.99 121.92 0)
+    (property "Footprint" "Capacitor_SMD:CP_Elec_6.3x7.7" (at 173.99 121.92 0)
       (effects (font (size 1.27 1.27)) hide)
     )
@@
       (effects (font (size 1.27 1.27)) (justify right))
     )
-    (property "Footprint" "" (at 341.63 123.19 0)
+    (property "Footprint" "Capacitor_SMD:CP_Elec_6.3x7.7" (at 341.63 123.19 0)
       (effects (font (size 1.27 1.27)) hide)
     )
@@
       (effects (font (size 1.27 1.27)) (justify right))
     )
-    (property "Footprint" "" (at 175.26 240.03 0)
-      (effects (font (size 1.27 1.27)) hide)
-    )
+    (property "Footprint" "Capacitor_SMD:CP_Elec_6.3x7.7" (at 175.26 240.03 0)
+      (effects (font (size 1.27 1.27)) hide)
+    )

Commit message: PCB Schematics finished
Parts:
- renumbered C22 to C401, C17 to C402, C23 to C403, C16 to C404, C24 to C405, C15 to C406, C25 to C407, C14 to C408, C48 to C409, C50 to C410, C49 to C411, C51 to C412, C18 to C413, C19 to C414, C20 to C415, C21 to C416, C46 to C417, C47 to C418, J6 to J401, J4 to J402, J7 to J403, J5 to J404, R23 to R403, R19 to R404, R24 to R405, R18 to R406, R25 to R407, R17 to R408, R20 to R410, R21 to R411, R22 to R412, T9 to T401, T10 to T402, T11 to T403, T12 to T404, T1 to T405, T2 to T406, T3 to T407, T4 to T408, T5 to T409, T6 to T410, T7 to T411, T8 to T412, U4 to U401, U2 to U402, U3 to U403

Commit message: Schematic updates
Parts:
- J401, J402, J404: footprint AMASS_XT60PW-F -> Connector_AMASS:AMASS_XT60PW-F_1x02_P7.20mm_Horizontal
- J403: footprint MSL Footprints:AMASS_XT60PW-M -> Connector_AMASS:AMASS_XT60PW-M_1x02_P7.20mm_Horizontal
Changed lines of the file:
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@@
       (effects (font (size 1.27 1.27)) (justify left))
     )
-    (property "Footprint" "AMASS_XT60PW-F" (at 181.61 82.55 0)
+    (property "Footprint" "Connector_AMASS:AMASS_XT60PW-F_1x02_P7.20mm_Horizontal" (at 181.61 82.55 0)
       (effects (font (size 1.27 1.27)) (justify bottom) hide)
     )
@@
       (effects (font (size 1.27 1.27)) (justify bottom) hide)
     )
-    (pin "S1")
-    (pin "S2")
     (pin "1")
     (pin "2")
@@
       (effects (font (size 1.27 1.27)) (justify left))
     )
-    (property "Footprint" "MSL Footprints:AMASS_XT60PW-M" (at 248.92 176.53 0)
+    (property "Footprint" "Connector_AMASS:AMASS_XT60PW-M_1x02_P7.20mm_Horizontal" (at 248.92 176.53 0)
       (effects (font (size 1.27 1.27)) (justify bottom) hide)
     )
@@
       (effects (font (size 1.27 1.27)) (justify left))
     )
-    (property "Footprint" "AMASS_XT60PW-F" (at 180.34 201.93 0)
+    (property "Footprint" "Connector_AMASS:AMASS_XT60PW-F_1x02_P7.20mm_Horizontal" (at 180.34 201.93 0)
       (effects (font (size 1.27 1.27)) (justify bottom) hide)
     )
@@
       (effects (font (size 1.27 1.27)) (justify bottom) hide)
     )
-    (pin "S1")
-    (pin "S2")
     (pin "1")
     (pin "2")
@@
       (effects (font (size 1.27 1.27)) (justify left))
     )
-    (property "Footprint" "AMASS_XT60PW-F" (at 349.25 82.55 0)
+    (property "Footprint" "Connector_AMASS:AMASS_XT60PW-F_1x02_P7.20mm_Horizontal" (at 349.25 82.55 0)
       (effects (font (size 1.27 1.27)) (justify bottom) hide)
     )
@@
       (effects (font (size 1.27 1.27)) (justify bottom) hide)
     )
-    (pin "S1")
-    (pin "S2")
-    (pin "1")
-    (pin "2")
+    (pin "1")
+    (pin "2")

Commit message: PCB layout progress, spice simulations for power board
Parts:
- added C419, C420, C421: 100u, Capacitor_SMD:CP_Elec_6.3x7.7, symbol Device:C_Polarized_Small
- added J405: XT60-M-Vertical, MSL Footprints:AMASS_XT60-M_1x02_P7.20mm_Vertical, symbol XT60PW-M:XT60-M-Vertical
- added J406, J407, J408: Conn_01x05, Connector_PinHeader_2.54mm:PinHeader_1x05_P2.54mm_Vertical, symbol Connector_Generic:Conn_01x05
- J401, J402, J404: footprint Connector_AMASS:AMASS_XT60PW-F_1x02_P7.20mm_Horizontal -> MSL Footprints:AMASS_XT60PW-F_1x02_P7.20mm_Horizontal
- J403: footprint Connector_AMASS:AMASS_XT60PW-M_1x02_P7.20mm_Horizontal -> MSL Footprints:AMASS_XT60PW-M_1x02_P7.20mm_Horizontal; now not fitted; now left out of the parts list
Connections:
- net GND: now also J403.1 (-), C419.2, C420.2, C421.2, J405.1 (-), J406.4 (Pin_4), J407.4 (Pin_4), J408.4 (Pin_4); no longer J403.2 (-)
- net VMOT: now also J403.2 (+), C419.1, C420.1, C421.1, J405.2 (+); no longer J403.1 (+)
- new net +3V3: J406.5 (Pin_5), J407.5 (Pin_5), J408.5 (Pin_5)
- new net SCL1: J406.3 (Pin_3)
- new net SCL2: J407.3 (Pin_3)
- new net SCL3: J408.3 (Pin_3)
- new net SDA1: J406.2 (Pin_2)
- new net SDA2: J407.2 (Pin_2)
- new net SDA3: J408.2 (Pin_2)

Commit message: Gateway board layout complete and routing begun
Parts:
- removed J406, J407, J408: Conn_01x05, Connector_PinHeader_2.54mm:PinHeader_1x05_P2.54mm_Vertical, symbol Connector_Generic:Conn_01x05
- added J406, J407, J409: JST_2.5mm_1x5, Connector_JST:JST_XH_B5B-XH-A_1x05_P2.50mm_Vertical, symbol MSL_Symbols:JST_2.5mm_1x5
Connections:
- net +3V3: now also J406.5 (Pin_5), J407.5 (Pin_5), J409.5 (Pin_5)
- net GND: now also J403.SH1, J406.4 (Pin_4), J407.4 (Pin_4), J409.4 (Pin_4)
- net SCL2: now also J406.3 (Pin_3)
- net SCL3: now also J407.3 (Pin_3)
- net SDA2: now also J406.2 (Pin_2)
- net SDA3: now also J407.2 (Pin_2)
- net VMOT: now also J403.SH2
- new net SCL4: J409.3 (Pin_3)
- new net SDA4: J409.2 (Pin_2)

Commit message: Sensor hub board done
Connections:
- net +3V3: now also R403.1, R404.1, R405.1, R406.1, R410.1, R411.1
- net M1_DVDD: no longer R404.1, R406.1
- net M2_DVDD: no longer R410.1, R411.1
- net M3_DVDD: no longer R403.1, R405.1
- no-connect marks 6 -> 12

Commit message: All boards done
Other:
- note added: "I_{DRIVE} = 100mA"
Changed lines of the file:
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@@
+    (effects (font (size 1.27 1.27)) (justify left bottom))
+  )
+  (text "I_{DRIVE} = 100mA" (at 248.92 113.03 0)
+    (effects (font (size 1.27 1.27)) (justify left bottom))
+  )
+  (text "I_{DRIVE} = 100mA" (at 81.28 113.03 0)
     (effects (font (size 1.27 1.27)) (justify left bottom))
   )
@@
     (effects (font (size 2.54 2.54)) (justify left bottom))
   )
+  (text "I_{DRIVE} = 100mA" (at 80.01 232.41 0)
+    (effects (font (size 1.27 1.27)) (justify left bottom))
+  )
   (text "16V Cap" (at 135.89 241.3 0)
