File: Electronics/Sensor Hub/Sensor Hub Board/sensors_connectors.kicad_sch (KiCad schematic)
At the start: 33 parts, among them J401 Conn_01x06_Pin, J402 Conn_01x06_Pin, J403 Conn_01x06_Pin, J404 Conn_01x06_Pin, J405 Conn_01x06_Pin, J406 Conn_01x06_Pin, J407 Conn_01x06_Pin, J408 Conn_01x06_Pin, J409 Conn_01x06_Pin, J410 Conn_01x06_Pin, J411 Conn_01x06_Pin, J412 Conn_01x06_Pin, J413 Conn_01x06_Pin, J414 Conn_01x06_Pin, J415 Conn_01x06_Pin, J416 Conn_01x06_Pin, U401 TCA9548APWR, U402 BMI270, U403 TCA9548APWR, U404 LIS3MDL

Commit message: Sensor hub board done
Parts:
- removed J401, J402, J403, J404, J405, J406, J407, J408, J409, J410, J411, J412, J413, J414, J415, J416: Conn_01x06_Pin, Connector_PinHeader_2.54mm:PinHeader_1x06_P2.54mm_Vertical, symbol Connector:Conn_01x06_Pin
- added J401, J402, J403, J404, J405, J406, J407, J408, J409, J410, J411, J412, J413, J414, J415, J416: JST_2.5mm_1x6, Connector_JST:JST_XH_B6B-XH-A_1x06_P2.50mm_Vertical, symbol MSL_Symbols:JST_2.5mm_1x6
- renumbered C406 to C402, C407 to C403, C403 to C404, C404 to C405, C402 to C406, C405 to C407
Connections:
- net GND: now also J401.2 (Pin_2), J402.2 (Pin_2), J403.2 (Pin_2), J404.2 (Pin_2), J405.2 (Pin_2), J406.2 (Pin_2), J407.2 (Pin_2), J408.2 (Pin_2), J409.2 (Pin_2), J410.2 (Pin_2), J411.2 (Pin_2), J412.2 (Pin_2), J413.2 (Pin_2), J414.2 (Pin_2), J415.2 (Pin_2), J416.2 (Pin_2)
- net GPIO0A: now also J401.5 (Pin_5)
- net GPIO0B: now also J401.6 (Pin_6)
- net GPIO10A: now also J404.5 (Pin_5)
- net GPIO10B: now also J404.6 (Pin_6)
- net GPIO11A: now also J408.5 (Pin_5)
- net GPIO11B: now also J408.6 (Pin_6)
- net GPIO12A: now also J411.5 (Pin_5)
- net GPIO12B: now also J411.6 (Pin_6)
- net GPIO13A: now also J415.5 (Pin_5)
- net GPIO13B: now also J415.6 (Pin_6)
- net GPIO14A: now also J412.5 (Pin_5)
- net GPIO14B: now also J412.6 (Pin_6)
- net GPIO15A: now also J416.5 (Pin_5)
- net GPIO15B: now also J416.6 (Pin_6)
- net GPIO1A: now also J405.5 (Pin_5)
- net GPIO1B: now also J405.6 (Pin_6)
- net GPIO2A: now also J402.5 (Pin_5)
- net GPIO2B: now also J402.6 (Pin_6)
- net GPIO3A: now also J406.5 (Pin_5)
- net GPIO3B: now also J406.6 (Pin_6)
- net GPIO4A: now also J409.5 (Pin_5)
- net GPIO5A: now also J413.5 (Pin_5)
- net GPIO5B: now also J413.6 (Pin_6)
- net GPIO6A: now also J410.5 (Pin_5)
- net GPIO6B: now also J410.6 (Pin_6)
- net GPIO7A: now also J414.5 (Pin_5)
- net GPIO7B: now also J414.6 (Pin_6)
- net GPIO8A: now also J403.5 (Pin_5)
- net GPIO8B: now also J403.6 (Pin_6)
- net GPIO9A: now also J407.5 (Pin_5)
- net GPIO9B: now also J407.6 (Pin_6)
- net SCL0: now also U401.18 (SC6), J401.3 (Pin_3); no longer U403.5 (SC0)
- net SCL1: now also U401.20 (SC7), J405.3 (Pin_3); no longer U403.7 (SC1)
- net SCL10: now also U403.20 (SC7), J404.3 (Pin_3); no longer U401.9 (SC2)
- net SCL11: now also U403.18 (SC6), J408.3 (Pin_3); no longer U401.11 (SC3)
- net SCL12: now also U403.16 (SC5), J411.3 (Pin_3); no longer U401.14 (SC4)
- net SCL13: now also U403.11 (SC3), J415.3 (Pin_3); no longer U401.16 (SC5)
- net SCL14: now also U403.14 (SC4), J412.3 (Pin_3); no longer U401.18 (SC6)
- net SCL15: now also U403.9 (SC2), J416.3 (Pin_3); no longer U401.20 (SC7)
- net SCL2: now also U401.5 (SC0), J402.3 (Pin_3); no longer U403.9 (SC2)
- net SCL3: now also U401.7 (SC1), J406.3 (Pin_3); no longer U403.11 (SC3)
- net SCL4: now also U401.9 (SC2), J409.3 (Pin_3); no longer U403.14 (SC4)
- net SCL5: now also U401.11 (SC3), J413.3 (Pin_3); no longer U403.16 (SC5)
- net SCL6: now also U401.16 (SC5), J410.3 (Pin_3); no longer U403.18 (SC6)
- net SCL7: now also U401.14 (SC4), J414.3 (Pin_3); no longer U403.20 (SC7)
- net SCL8: now also U403.7 (SC1), J403.3 (Pin_3); no longer U401.5 (SC0)
- net SCL9: now also U403.5 (SC0), J407.3 (Pin_3); no longer U401.7 (SC1)
- net SDA0: now also U401.17 (SD6), J401.4 (Pin_4); no longer U403.4 (SD0)
- net SDA1: now also U401.19 (SD7), J405.4 (Pin_4); no longer U403.6 (SD1)
- net SDA10: now also U403.19 (SD7), J404.4 (Pin_4); no longer U401.8 (SD2)
- net SDA11: now also U403.17 (SD6), J408.4 (Pin_4); no longer U401.10 (SD3)
- net SDA12: now also U403.15 (SD5), J411.4 (Pin_4); no longer U401.13 (SD4)
- net SDA13: now also U403.10 (SD3), J415.4 (Pin_4); no longer U401.15 (SD5)
- net SDA14: now also U403.13 (SD4), J412.4 (Pin_4); no longer U401.17 (SD6)
- net SDA15: now also U403.8 (SD2), J416.4 (Pin_4); no longer U401.19 (SD7)
- net SDA2: now also U401.4 (SD0), J402.4 (Pin_4); no longer U403.8 (SD2)
- net SDA3: now also U401.6 (SD1), J406.4 (Pin_4); no longer U403.10 (SD3)
- net SDA4: now also U401.8 (SD2), J409.4 (Pin_4); no longer U403.13 (SD4)
- net SDA5: now also U401.10 (SD3), J413.4 (Pin_4); no longer U403.15 (SD5)
- net SDA6: now also U401.15 (SD5), J410.4 (Pin_4); no longer U403.17 (SD6)
- net SDA7: now also U401.13 (SD4), J414.4 (Pin_4); no longer U403.19 (SD7)
- net SDA8: now also U403.6 (SD1), J403.4 (Pin_4); no longer U401.4 (SD0)
- net SDA9: now also U403.4 (SD0), J407.4 (Pin_4); no longer U401.6 (SD1)
- net VDDIO1: now also J401.1 (Pin_1), J402.1 (Pin_1), J405.1 (Pin_1), J406.1 (Pin_1)
- net VDDIO2: now also J409.1 (Pin_1), J410.1 (Pin_1), J413.1 (Pin_1), J414.1 (Pin_1)
- net VDDIO3: now also J403.1 (Pin_1), J404.1 (Pin_1), J407.1 (Pin_1), J408.1 (Pin_1)
- net VDDIO4: now also J411.1 (Pin_1), J412.1 (Pin_1), J415.1 (Pin_1), J416.1 (Pin_1)
- net SCL2_MCU renamed SCL4_MCU
- net SDA2_MCU renamed SDA4_MCU
- new net GPIO4B: J409.6 (Pin_6)
