File: Electronics/Sensor Hub/Sensor Hub Board/Sensor Hub Board.kicad_sch (KiCad schematic)
At the start: 4 parts

Commit message: PCB Schematics finished
Other:
- sheet Motor Drivers renamed Sensors & connectors
- sheet Sensors & connectors: file motor_driver.kicad_sch -> sensors_connectors.kicad_sch
Changed lines of the file:
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@@
     (pin "1")
     (instances
-      (project "Motor Driver Board"
+      (project "Sensor Hub Board"
         (path "/5318664d-e328-4e84-a383-7318275dc447"
           (reference "H104") (unit 1)
@@
     (pin "1")
     (instances
-      (project "Motor Driver Board"
+      (project "Sensor Hub Board"
         (path "/5318664d-e328-4e84-a383-7318275dc447"
           (reference "#PWR0104") (unit 1)
@@
     (pin "1")
     (instances
-      (project "Motor Driver Board"
+      (project "Sensor Hub Board"
         (path "/5318664d-e328-4e84-a383-7318275dc447"
           (reference "H102") (unit 1)
@@
     (pin "1")
     (instances
-      (project "Motor Driver Board"
+      (project "Sensor Hub Board"
         (path "/5318664d-e328-4e84-a383-7318275dc447"
           (reference "#PWR0103") (unit 1)
@@
     (pin "1")
     (instances
-      (project "Motor Driver Board"
+      (project "Sensor Hub Board"
         (path "/5318664d-e328-4e84-a383-7318275dc447"
           (reference "H103") (unit 1)
@@
     (pin "1")
     (instances
-      (project "Motor Driver Board"
+      (project "Sensor Hub Board"
         (path "/5318664d-e328-4e84-a383-7318275dc447"
           (reference "H101") (unit 1)
@@
     (pin "1")
     (instances
-      (project "Motor Driver Board"
+      (project "Sensor Hub Board"
         (path "/5318664d-e328-4e84-a383-7318275dc447"
           (reference "#PWR0101") (unit 1)
@@
     (pin "1")
     (instances
-      (project "Motor Driver Board"
+      (project "Sensor Hub Board"
         (path "/5318664d-e328-4e84-a383-7318275dc447"
           (reference "#PWR0102") (unit 1)
@@
     )
     (instances
-      (project "Motor Driver Board"
+      (project "Sensor Hub Board"
         (path "/5318664d-e328-4e84-a383-7318275dc447" (page "2"))
       )
@@
     )
     (instances
-      (project "Motor Driver Board"
+      (project "Sensor Hub Board"
         (path "/5318664d-e328-4e84-a383-7318275dc447" (page "3"))
       )
@@
     (stroke (width 0.1524) (type solid))
     (fill (color 0 0 194 1.0000))
-    (property "Sheetname" "Motor Drivers" (at 83.82 37.3884 0)
+    (property "Sheetname" "Sensors & connectors" (at 83.82 37.3884 0)
       (effects (font (size 1.27 1.27)) (justify left bottom))
     )
-    (property "Sheetfile" "motor_driver.kicad_sch" (at 83.82 79.3246 0)
+    (property "Sheetfile" "sensors_connectors.kicad_sch" (at 83.82 79.3246 0)
       (effects (font (size 1.27 1.27)) (justify left top))
     )
     (instances
-      (project "Motor Driver Board"
+      (project "Sensor Hub Board"
         (path "/5318664d-e328-4e84-a383-7318275dc447" (page "4"))
       )

Commit message: Sensor hub board done
Changed lines of the file:
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@@
+    (stroke (width 0) (type default))
+  )
+  (wire (pts (xy 81.28 111.76) (xy 81.28 114.3))
     (stroke (width 0) (type default))
   )
@@
     (stroke (width 0) (type default))
   )
+  (wire (pts (xy 74.93 114.3) (xy 74.93 111.76))
+    (stroke (width 0) (type default))
+  )
+  (wire (pts (xy 81.28 114.3) (xy 74.93 114.3))
+    (stroke (width 0) (type default))
+  )
   (symbol (lib_id "Mechanical:MountingHole_Pad") (at 57.15 119.38 0) (unit 1)
     (in_bom yes) (on_board yes) (dnp no) (fields_autoplaced)
@@
     )
   )
+  (symbol (lib_id "power:+3.3V") (at 74.93 111.76 0) (unit 1)
+    (in_bom yes) (on_board yes) (dnp no) (fields_autoplaced)
+    (property "Reference" "#PWR0105" (at 74.93 115.57 0)
+      (effects (font (size 1.27 1.27)) hide)
+    )
+    (property "Value" "+3.3V" (at 74.93 107.95 0)
+      (effects (font (size 1.27 1.27)))
+    )
+    (property "Footprint" "" (at 74.93 111.76 0)
+      (effects (font (size 1.27 1.27)) hide)
+    )
+    (property "Datasheet" "" (at 74.93 111.76 0)
+      (effects (font (size 1.27 1.27)) hide)
+    )
+    (pin "1")
+    (instances
+      (project "Sensor Hub Board"
+        (path "/5318664d-e328-4e84-a383-7318275dc447"
+          (reference "#PWR0105") (unit 1)
+        )
+      )
+      (project "Power Board"
+        (path "/d8843e0a-fd8a-4193-ba57-f0164156e030"
+          (reference "#PWR0105") (unit 1)
+        )
+      )
+    )
+  )
   (symbol (lib_id "power:GND") (at 57.15 106.68 0) (unit 1)
     (in_bom yes) (on_board yes) (dnp no) (fields_autoplaced)
@@
         )
       )
+    )
+  )
+  (symbol (lib_id "power:+3V3") (at 81.28 111.76 0) (unit 1)
+    (in_bom yes) (on_board yes) (dnp no) (fields_autoplaced)
+    (property "Reference" "#PWR0106" (at 81.28 115.57 0)
+      (effects (font (size 1.27 1.27)) hide)
+    )
+    (property "Value" "+3V3" (at 81.28 107.95 0)
+      (effects (font (size 1.27 1.27)))
+    )
+    (property "Footprint" "" (at 81.28 111.76 0)
+      (effects (font (size 1.27 1.27)) hide)
+    )
+    (property "Datasheet" "" (at 81.28 111.76 0)
+      (effects (font (size 1.27 1.27)) hide)
+    )
+    (pin "1")
+    (instances
+      (project "Sensor Hub Board"
+        (path "/5318664d-e328-4e84-a383-7318275dc447"
+          (reference "#PWR0106") (unit 1)
+        )
+      )
+      (project "Power Board"
+        (path "/d8843e0a-fd8a-4193-ba57-f0164156e030"
+          (reference "#PWR0106") (unit 1)
+        )
+      )

Commit message: All boards done
Connections:
- removed net GND: H101.1, H102.1, H103.1, H104.1
- no-connect marks 0 -> 4
Changed lines of the file:
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@@
 (kicad_sch (version 20230121) (generator eeschema)
   (paper "A5")
-  (wire (pts (xy 33.02 106.68) (xy 33.02 104.14))
-    (stroke (width 0) (type default))
-  )
-  (wire (pts (xy 57.15 106.68) (xy 57.15 104.14))
-    (stroke (width 0) (type default))
-  )
+  (no_connect (at 57.15 121.92))
+  (no_connect (at 57.15 104.14))
+  (no_connect (at 33.02 104.14))
+  (no_connect (at 33.02 121.92))
   (wire (pts (xy 81.28 111.76) (xy 81.28 114.3))
-    (stroke (width 0) (type default))
-  )
-  (wire (pts (xy 33.02 124.46) (xy 33.02 121.92))
-    (stroke (width 0) (type default))
-  )
-  (wire (pts (xy 57.15 124.46) (xy 57.15 121.92))
     (stroke (width 0) (type default))
   )
@@
         (path "/d8843e0a-fd8a-4193-ba57-f0164156e030"
           (reference "H4") (unit 1)
-        )
-      )
-    )
-  )
-  (symbol (lib_id "power:GND") (at 57.15 124.46 0) (unit 1)
-    (in_bom yes) (on_board yes) (dnp no) (fields_autoplaced)
-    (property "Reference" "#PWR0104" (at 57.15 130.81 0)
-      (effects (font (size 1.27 1.27)) hide)
-    )
-    (property "Value" "GND" (at 57.15 129.54 0)
-      (effects (font (size 1.27 1.27)))
-    )
-    (property "Footprint" "" (at 57.15 124.46 0)
-      (effects (font (size 1.27 1.27)) hide)
-    )
-    (property "Datasheet" "" (at 57.15 124.46 0)
-      (effects (font (size 1.27 1.27)) hide)
-    )
-    (pin "1")
-    (instances
-      (project "Sensor Hub Board"
-        (path "/5318664d-e328-4e84-a383-7318275dc447"
-          (reference "#PWR0104") (unit 1)
-        )
-      )
-      (project "Power Board"
-        (path "/d8843e0a-fd8a-4193-ba57-f0164156e030"
-          (reference "#PWR04") (unit 1)
         )
       )
@@
         (path "/d8843e0a-fd8a-4193-ba57-f0164156e030"
           (reference "#PWR0105") (unit 1)
-        )
-      )
-    )
-  )
-  (symbol (lib_id "power:GND") (at 57.15 106.68 0) (unit 1)
-    (in_bom yes) (on_board yes) (dnp no) (fields_autoplaced)
-    (property "Reference" "#PWR0103" (at 57.15 113.03 0)
-      (effects (font (size 1.27 1.27)) hide)
-    )
-    (property "Value" "GND" (at 57.15 111.76 0)
-      (effects (font (size 1.27 1.27)))
-    )
-    (property "Footprint" "" (at 57.15 106.68 0)
-      (effects (font (size 1.27 1.27)) hide)
-    )
-    (property "Datasheet" "" (at 57.15 106.68 0)
-      (effects (font (size 1.27 1.27)) hide)
-    )
-    (pin "1")
-    (instances
-      (project "Sensor Hub Board"
-        (path "/5318664d-e328-4e84-a383-7318275dc447"
-          (reference "#PWR0103") (unit 1)
-        )
-      )
-      (project "Power Board"
-        (path "/d8843e0a-fd8a-4193-ba57-f0164156e030"
-          (reference "#PWR03") (unit 1)
         )
       )
@@
         )
       )
-    )
-  )
-  (symbol (lib_id "power:GND") (at 33.02 106.68 0) (unit 1)
-    (in_bom yes) (on_board yes) (dnp no) (fields_autoplaced)
-    (property "Reference" "#PWR0101" (at 33.02 113.03 0)
-      (effects (font (size 1.27 1.27)) hide)
-    )
-    (property "Value" "GND" (at 33.02 111.76 0)
-      (effects (font (size 1.27 1.27)))
-    )
-    (property "Footprint" "" (at 33.02 106.68 0)
-      (effects (font (size 1.27 1.27)) hide)
-    )
-    (property "Datasheet" "" (at 33.02 106.68 0)
-      (effects (font (size 1.27 1.27)) hide)
-    )
-    (pin "1")
-    (instances
-      (project "Sensor Hub Board"
-        (path "/5318664d-e328-4e84-a383-7318275dc447"
-          (reference "#PWR0101") (unit 1)
-        )
-      )
-      (project "Power Board"
-        (path "/d8843e0a-fd8a-4193-ba57-f0164156e030"
-          (reference "#PWR01") (unit 1)
-        )
-      )
-    )
-  )
-  (symbol (lib_id "power:GND") (at 33.02 124.46 0) (unit 1)
-    (in_bom yes) (on_board yes) (dnp no) (fields_autoplaced)
-    (property "Reference" "#PWR0102" (at 33.02 130.81 0)
-      (effects (font (size 1.27 1.27)) hide)
-    )
-    (property "Value" "GND" (at 33.02 129.54 0)
-      (effects (font (size 1.27 1.27)))
-    )
-    (property "Footprint" "" (at 33.02 124.46 0)
-      (effects (font (size 1.27 1.27)) hide)
-    )
-    (property "Datasheet" "" (at 33.02 124.46 0)
-      (effects (font (size 1.27 1.27)) hide)
-    )
-    (pin "1")
-    (instances
-      (project "Sensor Hub Board"
-        (path "/5318664d-e328-4e84-a383-7318275dc447"
-          (reference "#PWR0102") (unit 1)
-        )
-      )
-      (project "Power Board"
-        (path "/d8843e0a-fd8a-4193-ba57-f0164156e030"
-          (reference "#PWR02") (unit 1)
-        )
-      )
