File: Electronics/Motors/Motor Encoder/Motor Encoder Board/Motor Encoder Board.kicad_sch (KiCad schematic)
At the start: 9 parts, among them IC1 AS5600L-ASOM, J1 Conn_01x05_Pin

Commit message: Sensor hub board done
Parts:
- removed J1: Conn_01x05_Pin, Connector_PinHeader_2.54mm:PinHeader_1x05_P2.54mm_Horizontal, symbol Connector:Conn_01x05_Pin
- added J1: JST_2.5mm_1x5, Connector_JST:JST_XH_B5B-XH-A_1x05_P2.50mm_Vertical, symbol MSL_Symbols:JST_2.5mm_1x5
Connections:
- net +3V3: now also J1.5 (Pin_5)
- net GND: now also J1.4 (Pin_4)
- net OUT: now also J1.1 (Pin_1)
- net SCL: now also J1.3 (Pin_3)
- net SDA: now also J1.2 (Pin_2)
Changed lines of the file:
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@@
+    )
+  )
+  (symbol (lib_id "MSL_Symbols:JST_2.5mm_1x5") (at 148.59 49.53 0) (mirror x) (unit 1)
+    (in_bom yes) (on_board yes) (dnp no) (fields_autoplaced)
+    (property "Reference" "J1" (at 148.59 39.37 0)
+      (effects (font (size 1.27 1.27)))
+    )
+    (property "Value" "JST_2.5mm_1x5" (at 148.59 41.91 0)
+      (effects (font (size 1.27 1.27)))
+    )
+    (property "Footprint" "Connector_JST:JST_XH_B5B-XH-A_1x05_P2.50mm_Vertical" (at 148.59 49.53 0)
+      (effects (font (size 1.27 1.27)) hide)
+    )
+    (property "Datasheet" "~" (at 148.59 49.53 0)
+      (effects (font (size 1.27 1.27)) hide)
+    )
+    (pin "1")
+    (pin "2")
+    (pin "3")
+    (pin "4")
+    (pin "5")
+    (instances
+      (project "Motor Encoder Board"
+        (path "/854825c0-4b52-484f-810c-81482f9ca65f"
+          (reference "J1") (unit 1)
+        )
+      )
     )
   )
   (symbol (lib_id "power:+3V3") (at 60.96 45.72 0) (unit 1)
     (in_bom yes) (on_board yes) (dnp no) (fields_autoplaced)
-    (property "Reference" "#PWR01" (at 60.96 49.53 0)
+    (property "Reference" "#PWR02" (at 60.96 49.53 0)
       (effects (font (size 1.27 1.27)) hide)
     )
@@
       (project "Motor Encoder Board"
         (path "/854825c0-4b52-484f-810c-81482f9ca65f"
-          (reference "#PWR01") (unit 1)
+          (reference "#PWR02") (unit 1)
         )
       )
@@
   (symbol (lib_id "power:+3V3") (at 124.46 36.83 0) (unit 1)
     (in_bom yes) (on_board yes) (dnp no) (fields_autoplaced)
-    (property "Reference" "#PWR04" (at 124.46 40.64 0)
+    (property "Reference" "#PWR07" (at 124.46 40.64 0)
       (effects (font (size 1.27 1.27)) hide)
     )
@@
       (project "Motor Encoder Board"
         (path "/854825c0-4b52-484f-810c-81482f9ca65f"
+          (reference "#PWR07") (unit 1)
+        )
+      )
+    )
+  )
+  (symbol (lib_id "power:GND") (at 86.36 90.17 0) (unit 1)
+    (in_bom yes) (on_board yes) (dnp no) (fields_autoplaced)
+    (property "Reference" "#PWR04" (at 86.36 96.52 0)
+      (effects (font (size 1.27 1.27)) hide)
+    )
+    (property "Value" "GND" (at 86.36 95.25 0)
+      (effects (font (size 1.27 1.27)))
+    )
+    (property "Footprint" "" (at 86.36 90.17 0)
+      (effects (font (size 1.27 1.27)) hide)
+    )
+    (property "Datasheet" "" (at 86.36 90.17 0)
+      (effects (font (size 1.27 1.27)) hide)
+    )
+    (pin "1")
+    (instances
+      (project "Motor Encoder Board"
+        (path "/854825c0-4b52-484f-810c-81482f9ca65f"
           (reference "#PWR04") (unit 1)
         )
@@
     )
   )
-  (symbol (lib_id "power:GND") (at 86.36 90.17 0) (unit 1)
-    (in_bom yes) (on_board yes) (dnp no) (fields_autoplaced)
-    (property "Reference" "#PWR06" (at 86.36 96.52 0)
-      (effects (font (size 1.27 1.27)) hide)
-    )
-    (property "Value" "GND" (at 86.36 95.25 0)
-      (effects (font (size 1.27 1.27)))
-    )
-    (property "Footprint" "" (at 86.36 90.17 0)
-      (effects (font (size 1.27 1.27)) hide)
-    )
-    (property "Datasheet" "" (at 86.36 90.17 0)
-      (effects (font (size 1.27 1.27)) hide)
-    )
-    (pin "1")
-    (instances
-      (project "Motor Encoder Board"
-        (path "/854825c0-4b52-484f-810c-81482f9ca65f"
-          (reference "#PWR06") (unit 1)
-        )
-      )
-    )
-  )
   (symbol (lib_id "power:GND") (at 140.97 58.42 0) (unit 1)
     (in_bom yes) (on_board yes) (dnp no) (fields_autoplaced)
-    (property "Reference" "#PWR07" (at 140.97 64.77 0)
+    (property "Reference" "#PWR08" (at 140.97 64.77 0)
       (effects (font (size 1.27 1.27)) hide)
     )
@@
       (project "Motor Encoder Board"
         (path "/854825c0-4b52-484f-810c-81482f9ca65f"
-          (reference "#PWR07") (unit 1)
+          (reference "#PWR08") (unit 1)
         )
       )
@@
   (symbol (lib_id "power:GND") (at 110.49 64.77 0) (unit 1)
     (in_bom yes) (on_board yes) (dnp no) (fields_autoplaced)
-    (property "Reference" "#PWR03" (at 110.49 71.12 0)
+    (property "Reference" "#PWR05" (at 110.49 71.12 0)
       (effects (font (size 1.27 1.27)) hide)
     )
@@
       (project "Motor Encoder Board"
         (path "/854825c0-4b52-484f-810c-81482f9ca65f"
-          (reference "#PWR03") (unit 1)
+          (reference "#PWR05") (unit 1)
         )
       )
@@
   (symbol (lib_id "power:GND") (at 58.42 90.17 0) (unit 1)
     (in_bom yes) (on_board yes) (dnp no) (fields_autoplaced)
-    (property "Reference" "#PWR08" (at 58.42 96.52 0)
+    (property "Reference" "#PWR01" (at 58.42 96.52 0)
       (effects (font (size 1.27 1.27)) hide)
     )
@@
       (project "Motor Encoder Board"
         (path "/854825c0-4b52-484f-810c-81482f9ca65f"
-          (reference "#PWR08") (unit 1)
+          (reference "#PWR01") (unit 1)
         )
       )
@@
         (path "/854825c0-4b52-484f-810c-81482f9ca65f"
           (reference "H1") (unit 1)
-        )
-      )
-    )
-  )
-  (symbol (lib_id "Connector:Conn_01x05_Pin") (at 148.59 49.53 180) (unit 1)
-    (in_bom yes) (on_board yes) (dnp no)
-    (property "Reference" "J1" (at 149.86 50.165 0)
-      (effects (font (size 1.27 1.27)) (justify right))
-    )
-    (property "Value" "Conn_01x05_Pin" (at 149.86 47.625 0)
-      (effects (font (size 1.27 1.27)) (justify right))
-    )
-    (property "Footprint" "Connector_PinHeader_2.54mm:PinHeader_1x05_P2.54mm_Horizontal" (at 148.59 49.53 0)
-      (effects (font (size 1.27 1.27)) hide)
-    )
-    (property "Datasheet" "~" (at 148.59 49.53 0)
-      (effects (font (size 1.27 1.27)) hide)
-    )
-    (pin "1")
-    (pin "2")
-    (pin "3")
-    (pin "4")
-    (pin "5")
-    (instances
-      (project "Motor Encoder Board"
-        (path "/854825c0-4b52-484f-810c-81482f9ca65f"
-          (reference "J1") (unit 1)
         )
       )
@@
   (symbol (lib_id "power:GND") (at 121.92 54.61 0) (unit 1)
     (in_bom yes) (on_board yes) (dnp no) (fields_autoplaced)
-    (property "Reference" "#PWR05" (at 121.92 60.96 0)
+    (property "Reference" "#PWR06" (at 121.92 60.96 0)
       (effects (font (size 1.27 1.27)) hide)
     )
@@
       (project "Motor Encoder Board"
         (path "/854825c0-4b52-484f-810c-81482f9ca65f"
-          (reference "#PWR05") (unit 1)
+          (reference "#PWR06") (unit 1)
         )
       )
@@
   (symbol (lib_id "power:GND") (at 60.96 55.88 0) (unit 1)
     (in_bom yes) (on_board yes) (dnp no) (fields_autoplaced)
-    (property "Reference" "#PWR02" (at 60.96 62.23 0)
+    (property "Reference" "#PWR03" (at 60.96 62.23 0)
       (effects (font (size 1.27 1.27)) hide)
     )
@@
       (project "Motor Encoder Board"
         (path "/854825c0-4b52-484f-810c-81482f9ca65f"
-          (reference "#PWR02") (unit 1)
-        )
-      )
+          (reference "#PWR03") (unit 1)
+        )
+      )

Commit message: All boards done
Connections:
- net GND: no longer H1.1, H2.1
- no-connect marks 0 -> 2
Changed lines of the file:
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@@
   (junction (at 71.12 54.61) (diameter 0) (color 0 0 0 0)
   )
+  (no_connect (at 86.36 87.63))
+  (no_connect (at 58.42 87.63))
   (wire (pts (xy 74.93 46.99) (xy 74.93 49.53))
     (stroke (width 0) (type default))
@@
     (stroke (width 0) (type default))
   )
-  (wire (pts (xy 58.42 90.17) (xy 58.42 87.63))
-    (stroke (width 0) (type default))
-  )
   (wire (pts (xy 107.95 52.07) (xy 133.35 52.07))
     (stroke (width 0) (type default))
@@
   )
   (wire (pts (xy 140.97 46.99) (xy 143.51 46.99))
-    (stroke (width 0) (type default))
-  )
-  (wire (pts (xy 86.36 90.17) (xy 86.36 87.63))
     (stroke (width 0) (type default))
   )
@@
     )
   )
-  (symbol (lib_id "power:GND") (at 86.36 90.17 0) (unit 1)
-    (in_bom yes) (on_board yes) (dnp no) (fields_autoplaced)
-    (property "Reference" "#PWR04" (at 86.36 96.52 0)
-      (effects (font (size 1.27 1.27)) hide)
-    )
-    (property "Value" "GND" (at 86.36 95.25 0)
-      (effects (font (size 1.27 1.27)))
-    )
-    (property "Footprint" "" (at 86.36 90.17 0)
-      (effects (font (size 1.27 1.27)) hide)
-    )
-    (property "Datasheet" "" (at 86.36 90.17 0)
-      (effects (font (size 1.27 1.27)) hide)
-    )
-    (pin "1")
-    (instances
-      (project "Motor Encoder Board"
-        (path "/854825c0-4b52-484f-810c-81482f9ca65f"
-          (reference "#PWR04") (unit 1)
-        )
-      )
-    )
-  )
   (symbol (lib_id "power:GND") (at 140.97 58.42 0) (unit 1)
     (in_bom yes) (on_board yes) (dnp no) (fields_autoplaced)
@@
         )
       )
-    )
-  )
-  (symbol (lib_id "power:GND") (at 58.42 90.17 0) (unit 1)
-    (in_bom yes) (on_board yes) (dnp no) (fields_autoplaced)
-    (property "Reference" "#PWR01" (at 58.42 96.52 0)
-      (effects (font (size 1.27 1.27)) hide)
-    )
-    (property "Value" "GND" (at 58.42 95.25 0)
-      (effects (font (size 1.27 1.27)))
-    )
-    (property "Footprint" "" (at 58.42 90.17 0)
-      (effects (font (size 1.27 1.27)) hide)
-    )
-    (property "Datasheet" "" (at 58.42 90.17 0)
-      (effects (font (size 1.27 1.27)) hide)
-    )
-    (pin "1")
-    (instances
-      (project "Motor Encoder Board"
-        (path "/854825c0-4b52-484f-810c-81482f9ca65f"
-          (reference "#PWR01") (unit 1)
-        )
-      )
