File: Electronics/Power/Power Board/Power Board.kicad_sch (KiCad schematic)
At the start: 4 parts

Commit message: All boards done
Connections:
- removed net GND: H101.1, H102.1, H103.1, H104.1
- no-connect marks 0 -> 4
Changed lines of the file:
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@@
 (kicad_sch (version 20230121) (generator eeschema)
   (paper "A5")
-  (wire (pts (xy 34.29 104.14) (xy 34.29 101.6))
-    (stroke (width 0) (type default))
-  )
+  (no_connect (at 34.29 119.38))
+  (no_connect (at 58.42 119.38))
+  (no_connect (at 34.29 101.6))
+  (no_connect (at 58.42 101.6))
   (wire (pts (xy 74.93 113.03) (xy 74.93 110.49))
     (stroke (width 0) (type default))
@@
   (wire (pts (xy 81.28 110.49) (xy 81.28 113.03))
     (stroke (width 0) (type default))
-  )
-  (wire (pts (xy 58.42 104.14) (xy 58.42 101.6))
-    (stroke (width 0) (type default))
-  )
-  (wire (pts (xy 34.29 121.92) (xy 34.29 119.38))
-    (stroke (width 0) (type default))
-  )
-  (wire (pts (xy 58.42 121.92) (xy 58.42 119.38))
-    (stroke (width 0) (type default))
-  )
-  (symbol (lib_id "power:GND") (at 34.29 121.92 0) (unit 1)
-    (in_bom yes) (on_board yes) (dnp no) (fields_autoplaced)
-    (property "Reference" "#PWR0102" (at 34.29 128.27 0)
-      (effects (font (size 1.27 1.27)) hide)
-    )
-    (property "Value" "GND" (at 34.29 127 0)
-      (effects (font (size 1.27 1.27)))
-    )
-    (property "Footprint" "" (at 34.29 121.92 0)
-      (effects (font (size 1.27 1.27)) hide)
-    )
-    (property "Datasheet" "" (at 34.29 121.92 0)
-      (effects (font (size 1.27 1.27)) hide)
-    )
-    (pin "1")
-    (instances
-      (project "Power Board"
-        (path "/d8843e0a-fd8a-4193-ba57-f0164156e030"
-          (reference "#PWR0102") (unit 1)
-        )
-      )
-    )
   )
   (symbol (lib_id "power:+3V3") (at 81.28 110.49 0) (unit 1)
@@
     )
   )
-  (symbol (lib_id "power:GND") (at 58.42 121.92 0) (unit 1)
-    (in_bom yes) (on_board yes) (dnp no) (fields_autoplaced)
-    (property "Reference" "#PWR0104" (at 58.42 128.27 0)
-      (effects (font (size 1.27 1.27)) hide)
-    )
-    (property "Value" "GND" (at 58.42 127 0)
-      (effects (font (size 1.27 1.27)))
-    )
-    (property "Footprint" "" (at 58.42 121.92 0)
-      (effects (font (size 1.27 1.27)) hide)
-    )
-    (property "Datasheet" "" (at 58.42 121.92 0)
-      (effects (font (size 1.27 1.27)) hide)
-    )
-    (pin "1")
-    (instances
-      (project "Power Board"
-        (path "/d8843e0a-fd8a-4193-ba57-f0164156e030"
-          (reference "#PWR0104") (unit 1)
-        )
-      )
-    )
-  )
   (symbol (lib_id "Mechanical:MountingHole_Pad") (at 58.42 116.84 0) (unit 1)
     (in_bom yes) (on_board yes) (dnp no) (fields_autoplaced)
@@
         )
       )
-    )
-  )
-  (symbol (lib_id "power:GND") (at 58.42 104.14 0) (unit 1)
-    (in_bom yes) (on_board yes) (dnp no) (fields_autoplaced)
-    (property "Reference" "#PWR0103" (at 58.42 110.49 0)
-      (effects (font (size 1.27 1.27)) hide)
-    )
-    (property "Value" "GND" (at 58.42 109.22 0)
-      (effects (font (size 1.27 1.27)))
-    )
-    (property "Footprint" "" (at 58.42 104.14 0)
-      (effects (font (size 1.27 1.27)) hide)
-    )
-    (property "Datasheet" "" (at 58.42 104.14 0)
-      (effects (font (size 1.27 1.27)) hide)
-    )
-    (pin "1")
-    (instances
-      (project "Power Board"
-        (path "/d8843e0a-fd8a-4193-ba57-f0164156e030"
-          (reference "#PWR0103") (unit 1)
-        )
-      )
-    )
-  )
-  (symbol (lib_id "power:GND") (at 34.29 104.14 0) (unit 1)
-    (in_bom yes) (on_board yes) (dnp no) (fields_autoplaced)
-    (property "Reference" "#PWR0101" (at 34.29 110.49 0)
-      (effects (font (size 1.27 1.27)) hide)
-    )
-    (property "Value" "GND" (at 34.29 109.22 0)
-      (effects (font (size 1.27 1.27)))
-    )
-    (property "Footprint" "" (at 34.29 104.14 0)
-      (effects (font (size 1.27 1.27)) hide)
-    )
-    (property "Datasheet" "" (at 34.29 104.14 0)
-      (effects (font (size 1.27 1.27)) hide)
-    )
-    (pin "1")
-    (instances
-      (project "Power Board"
-        (path "/d8843e0a-fd8a-4193-ba57-f0164156e030"
-          (reference "#PWR0101") (unit 1)
-        )
-      )
